File: hardware/kicad/module-I2C-Display_1_42inch.kicad_pcb (KiCad board)
At the start: 2 copper layers, 40 x 30 mm, 34 parts, among them J1 JST 4 Pin Qwiic I2C Connector, J2 JST 4 Pin Qwiic I2C Connector, J3 noknok_FlashPads_I2C-module, J4 noknok_UART_debug_1x3_pogo, Q1 2N7002, U1 CH32V003F4U6, U2 MT3540‑F23

Commit message: hardware: update KiCad layout and schematic, add BOM and schematic PDF
Parts:
- Q1: value 2N7002 -> 2N7002 or AO3400A (pin2pin)
- moved R5 18.1 mm to (128.4, 89.5), turned to 0 degrees
- moved D4 15.6 mm to (128.4, 84.8), turned to 180 degrees
- moved C9 5.88 mm to (141.3, 92.1), turned to 90 degrees
- moved C8 5.88 mm to (142.8, 92.1), turned to 90 degrees
- moved R7 5.77 mm to (141.1, 95.2), turned to -90 degrees
- moved R8 5.53 mm to (146.6, 86.7)
- moved Q1 5.34 mm to (143.7, 85.8)
- moved U2 5.02 mm to (127.9, 103.9)
- moved R6 4.84 mm to (139.6, 95.2), turned to -90 degrees
- moved L1 4.47 mm to (124.8, 103.3)
- moved C4 3.97 mm to (131.7, 92.0), turned to 180 degrees
- moved C2 3.34 mm to (133.3, 95.9), turned to -90 degrees
- moved D3 3.28 mm to (133.7, 105.4), turned to -90 degrees
- moved R9 3.20 mm to (140.7, 87.5)
- moved R2 2.99 mm to (131.7, 93.5), turned to 180 degrees
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Connections:
- U1 pad 10: Net-(DS1-RS/DC) -> Net-(DS1-RES)
- U1 pad 11: Net-(DS1-RES) -> Net-(DS1-RS/DC)
Routing:
- net +3.3V-PROT: track 77.4 -> 47.0 mm, vias 8 -> 5
- net GND: track 66.3 -> 85.3 mm, vias 48 -> 62
- net Net-(DS1-RS/DC): track 8.62 -> 19.3 mm
- net Net-(J1-Pin_4): track 36.9 -> 27.7 mm
- net Net-(DS1-SDA/MOSI): track 15.5 -> 6.42 mm
- net Net-(DS1-LEDK): track 16.3 -> 7.80 mm
- net +3.3V-IN: track 27.8 -> 34.3 mm
- net +4.5V: track 30.0 -> 36.1 mm
- net Net-(D3-A): track 4.81 -> 10.9 mm
- net Net-(J1-Pin_3): track 37.4 -> 42.3 mm
- net Net-(DS1-RES): track 25.0 -> 20.9 mm
- net Net-(Q1-G): track 9.13 -> 5.44 mm
- net Net-(DS1-SCL/SCK): track 4.74 -> 8.22 mm
- net Net-(D4-A): track 1.55 -> 4.78 mm
- net Net-(J4-TX): track 6.89 -> 9.16 mm
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Other:
- board text added: "1.42 inch 80x160 IPS Panel V2_Aug26"
- board text added: "UART Debug"
- board text removed: "1.42 inch 80x160 IPS Panel V1_Jun26"
- board text removed: "UART debug"
